File: _autosave-ccm.kicad_pcb (KiCad board)
At the start: 2 copper layers, 80.1 x 75.2 mm, 25 parts, among them J1 Conn_01x06_Socket, J2 Conn_01x06_Socket, J3 Conn_01x04_Socket, J4 Conn_01x04_Socket, J5 Conn_01x04_Socket, J6 Conn_01x02_Socket, J7 Conn_01x02_Socket, U1 Teensy4.1, U2 LM1117DT-1.8, U3 SN65HVD230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

Commit message: change brake and accel connectors
Changed lines of the file:
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@@
-	)
-	(segment
-		(start 137.76 77.68)
-		(end 137.76 77.76)
-		(width 0.2)
-		(layer "F.Cu")
-		(net 40)
 	)
 	(segment
@@
 		(width 0.2)
 		(layer "F.Cu")
-		(net 40)
-	)
-	(segment
-		(start 137.76 77.76)
-		(end 138 78)
-		(width 0.2)
-		(layer "F.Cu")
