File: ccm.kicad_pcb (KiCad board)
At the start: 2 copper layers, 125 x 100 mm, 88 parts, among them J1 Conn_01x02_Socket, J10 Conn_01x02_Socket, J11 Conn_01x02_Socket, J12 Conn_01x02_Socket, J13 Conn_01x02_Socket, J14 Conn_01x04_Socket, J15 Conn_01x02_Socket, J16 Conn_01x02_Socket, J17 Conn_01x04_Socket, J18 Conn_01x04_Socket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

Commit message: v2 fixes complete
Parts:
- removed J15, J24: Conn_01x02_Socket, Connector_Molex:Molex_Mini-Fit_Jr_5566-02A2_2x01_P4.20mm_Vertical
- removed Q4, Q5: MMBT3904, Package_TO_SOT_SMD:SOT-23
- removed R37: 10k, Resistor_SMD:R_0805_2012Metric
- removed R39: 1k, Resistor_SMD:R_0805_2012Metric
- added Q7: IRLZ34N, Package_TO_SOT_THT:TO-220-3_Vertical, F.Cu at (121.1, 87.7)
- added R24: 4.7k, Resistor_SMD:R_0805_2012Metric, F.Cu at (174.8, 71.8)
- added R45: 4.7k, Resistor_SMD:R_0805_2012Metric, F.Cu at (180.0, 71.8)
- J16: value Conn_01x02_Socket -> Conn_01x04_Socket; footprint Connector_Molex:Molex_Mini-Fit_Jr_5566-02A2_2x01_P4.20mm_Vertical -> Connector_Molex:Molex_Mini-Fit_Jr_5566-04A2_2x02_P4.20mm_Vertical
- moved J16 36.0 mm to (109.8, 87.2)
- moved R5 24.0 mm to (118.0, 141.0)
- moved R38 20.1 mm to (117.0, 89.7), turned to -90 degrees
- moved Q1 16.0 mm to (121.1, 135.9)
- moved J1 15.5 mm to (109.8, 138.2), turned to -90 degrees
- moved Q2 14.6 mm to (121.0, 120.3)
- moved Q3 14.6 mm to (121.0, 104.5)
- moved R33 14.6 mm to (126.2, 120.9)
- moved R34 14.6 mm to (126.2, 124.7)
- moved D1 14.6 mm to (116.1, 122.6)
- moved D2 14.6 mm to (116.0, 106.9)
- moved R35 14.6 mm to (126.2, 109.1)
- moved R36 14.6 mm to (126.2, 105.1)
- moved J11 14.6 mm to (109.8, 122.5)
- moved J12 14.6 mm to (109.8, 106.8)
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Connections:
- net Fan1+ renamed Fan+
- C1 pad 2: Pump1- -> GLV-
- C10 pad 1: Pump1- -> GLV-
- C2 pad 2: Pump1- -> GLV-
- C3 pad 2: Pump1- -> GLV-
- C4 pad 2: Pump1- -> GLV-
- C5 pad 2: Pump1- -> GLV-
- C6 pad 2: Pump1- -> GLV-
- C8 pad 2: Pump1- -> GLV-
- C9 pad 2: Pump1- -> GLV-
- D2 pad 2: Pump1- -> Pump2-
- J12 pad 2: Pump1- -> Pump2-
- J13 pad 2: Pump1- -> GLV-
- J14 pad 3: Pump1- -> GLV-
- J14 pad 4: Pump1- -> GLV-
- J16 pad 2: Pump1- -> Fan_PWM
- J17 pad 3: Pump1- -> GLV-
- J17 pad 4: Pump1- -> GLV-
- J18 pad 3: Pump1- -> GLV-
- J18 pad 4: Pump1- -> GLV-
- J5 pad 3: Pump1- -> GLV-
- J5 pad 4: Pump1- -> GLV-
- J6 pad 2: Pump1- -> GLV-
- Q1 pad 3: Pump1- -> GLV-
- Q2 pad 3: Pump1- -> GLV-
- Q3 pad 2: Pump1- -> Pump2-
- Q3 pad 3: Pump1- -> GLV-
- R11 pad 2: Pump1- -> GLV-
- R13 pad 2: Pump1- -> GLV-
- R15 pad 2: Pump1- -> GLV-
- R17 pad 2: Pump1- -> GLV-
- R19 pad 2: Pump1- -> GLV-
- R2 pad 2: Pump1- -> GLV-
- R21 pad 2: Pump1- -> GLV-
- R22 pad 1: Pump1- -> GLV-
- R29 pad 1: Pump1- -> GLV-
- R30 pad 1: Pump1- -> GLV-
- R34 pad 2: Pump1- -> GLV-
- R35 pad 2: Pump1- -> GLV-
- R38 pad 2: Fan2_PWM -> Fan_PWM
- R41 pad 2: +3.3V -> +5V
- R42 pad 2: +3.3V -> +5V
- R43 pad 2: +3.3V -> +5V
- R44 pad 2: +3.3V -> +5V
- R5 pad 1: Pump1- -> GLV-
- R7 pad 2: Pump1- -> GLV-
- U1 pad 1: Pump1- -> GLV-
- U1 pad 10: Net-(U1-8_TX2_IN1) -> unconnected-(U1-8_TX2_IN1-Pad10)
- U1 pad 47: Pump1- -> GLV-
- U2 pad 4: Pump1- -> GLV-
- U2 pad 7: Pump1- -> GLV-
- U3 pad 2: Pump1- -> GLV-
- U4 pad 2: Pump1- -> GLV-
- U5 pad 1: Pump1- -> GLV-
Routing:
- net Pump1-: track 324.2 -> 19.5 mm, vias 23 -> 0
- net GLV-: track 0.00 -> 89.1 mm, vias 0 -> 15
- net Net-(U1-8_TX2_IN1): track 39.1 -> 0.00 mm
- net Fan+: track 134.7 -> 97.7 mm
- net ready_to_drive_button: track 68.9 -> 102.8 mm, vias 1 -> 0
- net +5V: track 155.2 -> 186.2 mm, vias 0 -> 2
- net +3.3V: track 74.6 -> 44.6 mm, vias 2 -> 1
- net speaker_pwm: track 20.3 -> 42.8 mm, vias 2 -> 1
- net Net-(Q1-G): track 37.2 -> 59.7 mm, vias 2 -> 1
- net Fan2_PWM: track 21.4 -> 0.00 mm
- net Pump2-: track 0.00 -> 19.2 mm
- net Fan_PWM: track 0.00 -> 11.7 mm
- net PWM_in_2: track 10.4 -> 19.5 mm
- net Net-(U1-7_RX2_OUT1A): track 34.7 -> 25.9 mm
- net Net-(U1-26_A12_MOSI1): track 38.7 -> 30.4 mm
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- added copper zone on B.Cu, net GLV-
- added copper zone on F.Cu, net GLV-
- removed copper zone on B.Cu, net Pump1-
- removed copper zone on F.Cu, net Pump1-
Other:
- board text added: "24V IN"
- board text added: "ACCEL/BRAKE PEDAL"
- board text added: "BRAKE LIGHT/RTM"
- board text added: "CAN1"
- board text added: "CAN2"
- board text added: "FANS"
- board text added: "GPIO 1/2"
- board text added: "GPIO 3/4"
- board text added: "I2C"
- board text added: "LINEAR POTS"
- board text added: "POWER IN"
- board text added: "PUMP1"
- board text added: "PUMP2"
- board text added: "SPEAKER"
- board text added: "THERMISTOR 1/2"
- board text added: "THERMISTOR 3/4"
- board text added: "WHEEL PWM"
