File: ccm.kicad_sch (KiCad schematic)
At the start: 88 parts, among them J1 Conn_01x02_Socket, J10 Conn_01x02_Socket, J11 Conn_01x02_Socket, J12 Conn_01x02_Socket, J13 Conn_01x02_Socket, J14 Conn_01x04_Socket, J15 Conn_01x02_Socket, J16 Conn_01x02_Socket, J17 Conn_01x04_Socket, J18 Conn_01x04_Socket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

Commit message: v2 fixes complete
Parts:
- removed J15, J16, J24: Conn_01x02_Socket, Connector_Molex:Molex_Mini-Fit_Jr_5566-02A2_2x01_P4.20mm_Vertical, symbol Connector:Conn_01x02_Socket
- removed Q4, Q5: MMBT3904, Package_TO_SOT_SMD:SOT-23, symbol Transistor_BJT:MMBT3904
- removed R37: 10k, Resistor_SMD:R_0805_2012Metric, symbol Device:R_US
- removed R39: 1k, Resistor_SMD:R_0805_2012Metric, symbol Device:R_US
- added J16: Conn_01x04_Socket, Connector_Molex:Molex_Mini-Fit_Jr_5566-04A2_2x02_P4.20mm_Vertical, symbol Connector:Conn_01x04_Socket
- added Q7: IRLZ34N, Package_TO_SOT_THT:TO-220-3_Vertical, symbol Transistor_FET:IRLZ34N
- added R24, R45: 4.7k, Resistor_SMD:R_0805_2012Metric, symbol Device:R_US
Connections:
- net +24V: now also J16.1 (Pin_1)
- net +3.3V: no longer R41.2, R42.2, R43.2, R44.2
- net +5V: now also R41.2, R42.2, R43.2, R44.2, R24.2, R45.2
- net GLV-: now also J16.3 (Pin_3), Q7.3 (S); no longer D1.2 (A), D2.2 (A), J11.2 (Pin_2), J12.2 (Pin_2), Q2.2 (D), Q3.2 (D)
- net PWM_in_1: now also R45.1
- net PWM_in_2: now also R24.1
- net at R40.1: now also Q7.1 (G)
- net Fan2_PWM renamed Fan_PWM
- net Fan_PWM: now also J16.2 (Pin_2), Q7.2 (D)
- new net Pump1-: D1.2 (A), J11.2 (Pin_2), Q2.2 (D)
- new net Pump2-: D2.2 (A), J12.2 (Pin_2), Q3.2 (D)
- no-connect marks 25 -> 33
Other:
- note added: "Fan Output"
- note added: "Pump Output"
- note removed: "Fan PWM OUT"
- note removed: "Pump/Fan Output"
- moved on the sheet: R22
